Commit message: second commit

File: urdf/iiwa7.urdf (robot description, URDF)
Before this commit: robot iiwa7_robot, 8 links, 7 joints
Links:
- link end_effector: geometry collision cylinder length=0.05 radius=0.06; visual box size=0.06 0.06 0.07

Commit message: fixed urdf

File: urdf/iiwa7.urdf (robot description, URDF)
Before this commit: robot iiwa7_robot, 8 links, 7 joints
Links:
- link end_effector: geometry collision box size=0.06 0.06 0.07; visual box size=0.06 0.06 0.07
